File: board/PicoParanoia.kicad_sch (KiCad schematic)
At the start: 62 parts, among them J1 RCAJack, J2 Barrel_Jack_Switch, J3 Conn_01x04_Pin, J4 DE9_Plug, P1 Mini-DIN_6pins_ver4, Q1 2N3904, Q2 2N3904, Q3 2N3904, Q4 2N3904, U1 MicroSD_SPI_CD, U2 Pico, U3 MicroSD_SPI_CD, U4 LM7805_TO220, U5 NE555D, U6 MAX232

Commit message: Change R1/R2 from 10R to 0R (power supply isolation fix)
Fixes the marginal SD card init failures traced to Vcc sag during the
current-hungry card init sequence.

Co-Authored-By: Claude Opus 4.8 <noreply@anthropic.com>
Parts:
- R1, R2: value 10R -> 0R
Changed lines of the file:
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@@
       (effects (font (size 1.27 1.27)) (justify left))
     )
-    (property "Value" "10R" (at 199.39 35.56 90)
+    (property "Value" "0R" (at 199.39 34.925 90)
       (effects (font (size 1.27 1.27)) (justify left))
     )
@@
       (effects (font (size 1.27 1.27)) (justify left))
     )
-    (property "Value" "10R" (at 156.21 36.83 90)
-      (effects (font (size 1.27 1.27)) (justify left))
-    )
+    (property "Value" "0R" (at 156.21 36.068 90)
+      (effects (font (size 1.27 1.27)) (justify left))
+    )
